Commit message: Add ros_control to simulation

File: carpincho_description/urdf/include/common_macros.urdf.xacro (robot description, xacro)
@@ -62,4 +62,5 @@
       <child link="${prefix}_wheel"/>
       <origin xyz="${pos_x_joint} ${reflect* pos_y_joint} ${pos_z_joint}" rpy="0 0 0"/>
+      <dynamics damping="0.0" friction="4.5"/>
     </joint>
     <transmission name="${prefix}_wheel_transmission">

File: carpincho_simulation/urdf/carpincho.gazebo.xacro (robot description, xacro)
@@ -14,11 +14,12 @@
   <xacro:friction reference="front_right_wheel" mu="100"/>
   <xacro:friction reference="front_left_wheel" mu="100"/>
-  <xacro:friction reference="rear_caster_base_link" mu="0.05"/>
-<!-- ROS Control not supported(yet)  -->
-  <!--
+  <xacro:friction reference="rear_caster_wheel_link" mu="0.05"/>
   <gazebo>
     <plugin name="gazebo_ros_control" filename="libgazebo_ros_control.so">
+        <!-- <robotNamespace>: The ROS namespace to be used for this instance of the plugin, defaults to robot name in URDF/SDF -->
+        <!-- <controlPeriod>: The period of the controller update (in seconds), defaults to Gazebo's period -->
+        <!-- <robotParam>: The location of the robot_description (URDF) on the parameter server, defaults to /robot_description' -->
+        <!-- <robotSimType>: The pluginlib name of a custom robot sim interface to be used, defaults to 'DefaultRobotHWSim' -->
     </plugin>
   </gazebo>
-  -->
 </robot>
