Commit message: Adds camera to the robot.
Signed-off-by: Franco Cipollone <franco.c@ekumenlabs.com>

File: carpincho_description/urdf/carpincho.urdf.xacro (robot description, xacro)
@@ -58,4 +58,6 @@
                    sensor_prop="${sensor_prop}">
   </xacro:laser>
+  <xacro:camera_sensor parent_link="base_link" sensor_prop="${sensor_prop}">
+  </xacro:camera_sensor>
   <!-- ros2_control -->
   <xacro:include filename="$(find ${package_name})/urdf/include/carpincho_control.urdf.xacro" />

File: carpincho_description/urdf/include/common_sensors.urdf.xacro (robot description, xacro)
@@ -42,3 +42,45 @@
   </joint>
 </xacro:macro>
+<xacro:macro name="camera_sensor" params="parent_link sensor_prop">
+  <xacro:property name="mesh"
+     value="${sensor_prop['camera']['mesh']}"/>
+  <link name="camera_link">
+    <xacro:if value="${mesh != '' }" >
+      <visual>
+        <origin xyz="0 0 0" rpy="0 0 0"/>
+        <geometry>
+          <mesh filename="package://${package_name}/meshes/sensors/${mesh}" />
+        </geometry>
+        <material name="blue"/>
+      </visual>
+    </xacro:if>
+    <xacro:if value="${mesh == '' }" >
+      <visual>
+        <origin xyz="0 0 0" rpy="0 0 0"/>
+        <geometry>
+          <box size="${sensor_prop['camera']['box_size']} ${sensor_prop['camera']['box_size']} ${sensor_prop['camera']['box_size']}"/>
+        </geometry>
+        <material name="blue"/>
+      </visual>
+    </xacro:if>
+    <collision>
+      <origin xyz="0 0 0" rpy="0 0 0"/>
+      <geometry>
+        <box size="${sensor_prop['camera']['box_size']} ${sensor_prop['camera']['box_size']} ${sensor_prop['camera']['box_size']}"/>
+      </geometry>
+    </collision>
+    <xacro:box_inertia m="${sensor_prop['camera']['mass']}"
+                            x="${sensor_prop['camera']['box_size']}"
+                            y="${sensor_prop['camera']['box_size']}"
+                            z="${sensor_prop['camera']['box_size']}"
+                            o_xyz="0 0 0"
+                            o_rpy="0 0 0" />
+  </link>
+  <joint name="camera_joint" type="fixed">
+    <parent link="${parent_link}"/>
+    <child link="camera_link"/>
+    <origin xyz="${sensor_prop['camera']['dx']} ${sensor_prop['camera']['dy']} ${sensor_prop['camera']['dz']}" rpy="0 0 0"/>
+    <axis xyz="0 1 0" />
+  </joint>
+</xacro:macro>
 </robot>
