Commit message: Updates motor colors.
Signed-off-by: Franco Cipollone <franco.c@ekumenlabs.com>

File: andino_description/urdf/include/common_macros.urdf.xacro (robot description, xacro)
@@ -90,5 +90,5 @@
           </xacro:if>
         </geometry>
-        <material name="yellow"/>
+        <material name="light_blue"/>
       </visual>
     </xacro:if>
@@ -252,5 +252,5 @@
   </material>
   <material name="light_blue">
-    <color rgba="0 0.9 1.0 1"/>
+    <color rgba="0 0.5 0.8 1"/>
   </material>
   <material name="black">
