Commit message: Hardware configuration is now being loaded from YAML file, updated README and updated launch files to pass xacro arguments
Signed-off-by: JesusSilvaUtrera <jsilvautrera@gmail.com>

File: andino_description/urdf/include/andino_control.urdf.xacro (robot description, xacro)
@@ -1,32 +1,37 @@
 <?xml version="1.0"?>
 <robot xmlns:xacro="http://www.ros.org/wiki/xacro">
-  <!-- TODO(francocipollone): This xacro should be part of andino_control package instead.-->
-  <ros2_control name="RealRobot" type="system">
-    <hardware>
-      <plugin>andino_base/DiffDriveAndino</plugin>
-      <!-- TODO(francocipollone): Parameters like loop_rate, device, baud_rate, etc should be loaded from a file or passed via the launch file as xacro args -->
-      <param name="left_wheel_name">left_wheel_joint</param>
-      <param name="right_wheel_name">right_wheel_joint</param>
-      <param name="serial_device">/dev/ttyUSB_ARDUINO</param>
-      <param name="baud_rate">57600</param>
-      <param name="timeout">1000</param>
-      <param name="enc_ticks_per_rev">585</param>
-    </hardware>
-    <joint name="left_wheel_joint">
-      <command_interface name="velocity">
-        <param name="min">-5</param>
-        <param name="max">5</param>
-      </command_interface>
-      <state_interface name="velocity"/>
-      <state_interface name="position"/>
-    </joint>
-    <joint name="right_wheel_joint">
-      <command_interface name="velocity">
-        <param name="min">-5</param>
-        <param name="max">5</param>
-      </command_interface>
-      <state_interface name="velocity"/>
-      <state_interface name="position"/>
-    </joint>
-  </ros2_control>
+<!-- ===================== Control xacro =========================================
+  params:
+  - hardware_props [dictionary]: hardware properties loaded from the YAML file.
+-->
+  <xacro:macro name="control" params="hardware_props" >
+    <!-- TODO(francocipollone): This xacro should be part of andino_control package instead.-->
+    <ros2_control name="RealRobot" type="system">
+      <hardware>
+        <plugin>andino_base/DiffDriveAndino</plugin>
+        <param name="left_wheel_name">left_wheel_joint</param>
+        <param name="right_wheel_name">right_wheel_joint</param>
+        <param name="serial_device">/dev/ttyUSB_ARDUINO</param>
+        <param name="baud_rate">57600</param>
+        <param name="timeout">1000</param>
+        <param name="enc_ticks_per_rev">585</param>
+      </hardware>
+      <joint name="left_wheel_joint">
+        <command_interface name="velocity">
+          <param name="min">-5</param>
+          <param name="max">5</param>
+        </command_interface>
+        <state_interface name="velocity"/>
+        <state_interface name="position"/>
+      </joint>
+      <joint name="right_wheel_joint">
+        <command_interface name="velocity">
+          <param name="min">-5</param>
+          <param name="max">5</param>
+        </command_interface>
+        <state_interface name="velocity"/>
+        <state_interface name="position"/>
+      </joint>
+    </ros2_control>
+  </xacro:macro>
 </robot>
