Commit message: Gazebo Classic Simulation humble (#78)
Gazebo classic simulation of Andino in ros 2.
---------

Signed-off-by: olmerg <olmerg@gmail.com>

File: andino_description/urdf/include/common_sensors.urdf.xacro (robot description, xacro)
@@ -50,5 +50,5 @@
         <origin xyz="0 0 0" rpy="0 0 0"/>
         <geometry>
-          <mesh filename="package://${package_name}/meshes/sensors/${mesh}" />
+          <mesh filename="package://andino_description/meshes/sensors/${mesh}" />
         </geometry>
         <material name="blue"/>

Commit message: Update sensors urdf.
Signed-off-by: Miguel <miguel.diaz@creativa77.com.ar>

File: andino_description/urdf/include/common_sensors.urdf.xacro (robot description, xacro)
@@ -48,5 +48,5 @@
     <xacro:if value="${mesh != '' }" >
       <visual>
-        <origin xyz="0 0 0" rpy="0 0 0"/>
+        <origin xyz="0 0 0" rpy="${pi/2} 0 ${-pi/2}"/>
         <geometry>
           <mesh filename="package://andino_description/meshes/sensors/${mesh}" />
