Commit message: One Andino with diff_drive plugin
Signed-off-by: olmerg <olmerg@gmail.com>

File: andino_description/urdf/include/andino_caster_macro.urdf.xacro (robot description, xacro)
@@ -28,8 +28,8 @@
           <geometry>
             <xacro:if value="${scale != '' }" >
-              <mesh filename="package://andino_description/meshes/${robot_name}/${wheel_props['base']['mesh']}" scale="${scale}"/>
+              <mesh filename="file://$(find andino_description)/meshes/${robot_name}/${wheel_props['base']['mesh']}" scale="${scale}"/>
             </xacro:if>
             <xacro:if value="${scale == '' }" >
-              <mesh filename="package://andino_description/meshes/${robot_name}/${wheel_props['base']['mesh']}" />
+              <mesh filename="file://$(find andino_description)/meshes/${robot_name}/${wheel_props['base']['mesh']}" />
             </xacro:if>
           </geometry>
@@ -74,8 +74,8 @@
           <geometry>
             <xacro:if value="${scale != '' }" >
-              <mesh filename="package://andino_description/meshes/${robot_name}/${wheel_props['hub']['mesh']}" scale="${scale}"/>
+              <mesh filename="file://$(find andino_description)/meshes/${robot_name}/${wheel_props['hub']['mesh']}" scale="${scale}"/>
             </xacro:if>
             <xacro:if value="${scale == '' }" >
-              <mesh filename="package://andino_description/meshes/${robot_name}/${wheel_props['hub']['mesh']}" />
+              <mesh filename="file://$(find andino_description)/meshes/${robot_name}/${wheel_props['hub']['mesh']}" />
             </xacro:if>
           </geometry>
@@ -118,8 +118,8 @@
           <geometry>
             <xacro:if value="${scale != '' }" >
-              <mesh filename="package://andino_description/meshes/${robot_name}/${wheel_props['wheel']['mesh']}" scale="${scale}"/>
+              <mesh filename="file://$(find andino_description)/meshes/${robot_name}/${wheel_props['wheel']['mesh']}" scale="${scale}"/>
             </xacro:if>
             <xacro:if value="${scale == '' }" >
-              <mesh filename="package://andino_description/meshes/${robot_name}/${wheel_props['wheel']['mesh']}" />
+              <mesh filename="file://$(find andino_description)/meshes/${robot_name}/${wheel_props['wheel']['mesh']}" />
             </xacro:if>
           </geometry>

File: andino_description/urdf/include/common_macros.urdf.xacro (robot description, xacro)
@@ -23,8 +23,8 @@
         <geometry>
           <xacro:if value="${wheel_props['scale'] == '' }" >
-            <mesh filename="package://andino_description/meshes/${robot_name}/${wheel_props['mesh']}" />
+            <mesh filename="file://$(find andino_description)/meshes/${robot_name}/${wheel_props['mesh']}" />
           </xacro:if>
           <xacro:if value="${wheel_props['scale'] == '' }" >
-            <mesh filename="package://andino_description/meshes/${robot_name}/${wheel_props['mesh']}" scale="${wheel_props['scale']}" />
+            <mesh filename="file://$(find andino_description)/meshes/${robot_name}/${wheel_props['mesh']}" scale="${wheel_props['scale']}" />
           </xacro:if>
         </geometry>
@@ -84,8 +84,8 @@
         <geometry>
           <xacro:if value="${motor_props['scale'] == '' }" >
-            <mesh filename="package://andino_description/meshes/${robot_name}/${motor_props['mesh']}" />
+            <mesh filename="file://$(find andino_description)/meshes/${robot_name}/${motor_props['mesh']}" />
           </xacro:if>
           <xacro:if value="${motor_props['scale'] != '' }" >
-            <mesh filename="package://andino_description/meshes/${robot_name}/${motor_props['mesh']}" scale="${motor_props['scale']}"/>
+            <mesh filename="file://$(find andino_description)/meshes/${robot_name}/${motor_props['mesh']}" scale="${motor_props['scale']}"/>
           </xacro:if>
         </geometry>
@@ -143,8 +143,8 @@
           <!-- The folder path get a folder_name global parameter -->
           <xacro:if value="${scale != '' }" >
-            <mesh filename="package://andino_description/meshes/${robot_name}/${mesh}" scale="${scale}"/>
+            <mesh filename="file://$(find andino_description)/meshes/${robot_name}/${mesh}" scale="${scale}"/>
           </xacro:if>
           <xacro:if value="${scale == '' }" >
-            <mesh filename="package://andino_description/meshes/${robot_name}/${mesh}" />
+            <mesh filename="file://$(find andino_description)/meshes/${robot_name}/${mesh}" />
           </xacro:if>
         </geometry>

Commit message: One Andino with diff_drive plugin
Signed-off-by: olmerg <olmerg@gmail.com>

File: andino_description/urdf/include/andino_caster_macro.urdf.xacro (robot description, xacro)
@@ -28,8 +28,8 @@
           <geometry>
             <xacro:if value="${scale != '' }" >
-              <mesh filename="package://andino_description/meshes/${robot_name}/${wheel_props['base']['mesh']}" scale="${scale}"/>
+              <mesh filename="file://$(find andino_description)/meshes/${robot_name}/${wheel_props['base']['mesh']}" scale="${scale}"/>
             </xacro:if>
             <xacro:if value="${scale == '' }" >
-              <mesh filename="package://andino_description/meshes/${robot_name}/${wheel_props['base']['mesh']}" />
+              <mesh filename="file://$(find andino_description)/meshes/${robot_name}/${wheel_props['base']['mesh']}" />
             </xacro:if>
           </geometry>
@@ -74,8 +74,8 @@
           <geometry>
             <xacro:if value="${scale != '' }" >
-              <mesh filename="package://andino_description/meshes/${robot_name}/${wheel_props['hub']['mesh']}" scale="${scale}"/>
+              <mesh filename="file://$(find andino_description)/meshes/${robot_name}/${wheel_props['hub']['mesh']}" scale="${scale}"/>
             </xacro:if>
             <xacro:if value="${scale == '' }" >
-              <mesh filename="package://andino_description/meshes/${robot_name}/${wheel_props['hub']['mesh']}" />
+              <mesh filename="file://$(find andino_description)/meshes/${robot_name}/${wheel_props['hub']['mesh']}" />
             </xacro:if>
           </geometry>
@@ -118,8 +118,8 @@
           <geometry>
             <xacro:if value="${scale != '' }" >
-              <mesh filename="package://andino_description/meshes/${robot_name}/${wheel_props['wheel']['mesh']}" scale="${scale}"/>
+              <mesh filename="file://$(find andino_description)/meshes/${robot_name}/${wheel_props['wheel']['mesh']}" scale="${scale}"/>
             </xacro:if>
             <xacro:if value="${scale == '' }" >
-              <mesh filename="package://andino_description/meshes/${robot_name}/${wheel_props['wheel']['mesh']}" />
+              <mesh filename="file://$(find andino_description)/meshes/${robot_name}/${wheel_props['wheel']['mesh']}" />
             </xacro:if>
           </geometry>

Commit message: from file to package in the xacro
Signed-off-by: olmerg <olmerg@gmail.com>

File: andino_description/urdf/include/andino_caster_macro.urdf.xacro (robot description, xacro)
@@ -28,8 +28,8 @@
           <geometry>
             <xacro:if value="${scale != '' }" >
-              <mesh filename="file://$(find andino_description)/meshes/${robot_name}/${wheel_props['base']['mesh']}" scale="${scale}"/>
+              <mesh filename="package://andino_description/meshes/${robot_name}/${wheel_props['base']['mesh']}" scale="${scale}"/>
             </xacro:if>
             <xacro:if value="${scale == '' }" >
-              <mesh filename="file://$(find andino_description)/meshes/${robot_name}/${wheel_props['base']['mesh']}" />
+              <mesh filename="package://andino_description/meshes/${robot_name}/${wheel_props['base']['mesh']}" />
             </xacro:if>
           </geometry>
@@ -74,8 +74,8 @@
           <geometry>
             <xacro:if value="${scale != '' }" >
-              <mesh filename="file://$(find andino_description)/meshes/${robot_name}/${wheel_props['hub']['mesh']}" scale="${scale}"/>
+              <mesh filename="package://andino_description/meshes/${robot_name}/${wheel_props['hub']['mesh']}" scale="${scale}"/>
             </xacro:if>
             <xacro:if value="${scale == '' }" >
-              <mesh filename="file://$(find andino_description)/meshes/${robot_name}/${wheel_props['hub']['mesh']}" />
+              <mesh filename="package://andino_description/meshes/${robot_name}/${wheel_props['hub']['mesh']}" />
             </xacro:if>
           </geometry>
@@ -118,8 +118,8 @@
           <geometry>
             <xacro:if value="${scale != '' }" >
-              <mesh filename="file://$(find andino_description)/meshes/${robot_name}/${wheel_props['wheel']['mesh']}" scale="${scale}"/>
+              <mesh filename="package://andino_description/meshes/${robot_name}/${wheel_props['wheel']['mesh']}" scale="${scale}"/>
             </xacro:if>
             <xacro:if value="${scale == '' }" >
-              <mesh filename="file://$(find andino_description)/meshes/${robot_name}/${wheel_props['wheel']['mesh']}" />
+              <mesh filename="package://andino_description/meshes/${robot_name}/${wheel_props['wheel']['mesh']}" />
             </xacro:if>
           </geometry>

File: andino_description/urdf/include/common_macros.urdf.xacro (robot description, xacro)
@@ -23,8 +23,8 @@
         <geometry>
           <xacro:if value="${wheel_props['scale'] == '' }" >
-            <mesh filename="file://$(find andino_description)/meshes/${robot_name}/${wheel_props['mesh']}" />
+            <mesh filename="package://andino_description/meshes/${robot_name}/${wheel_props['mesh']}" />
           </xacro:if>
           <xacro:if value="${wheel_props['scale'] == '' }" >
-            <mesh filename="file://$(find andino_description)/meshes/${robot_name}/${wheel_props['mesh']}" scale="${wheel_props['scale']}" />
+            <mesh filename="package://andino_description/meshes/${robot_name}/${wheel_props['mesh']}" scale="${wheel_props['scale']}" />
           </xacro:if>
         </geometry>
@@ -84,8 +84,8 @@
         <geometry>
           <xacro:if value="${motor_props['scale'] == '' }" >
-            <mesh filename="file://$(find andino_description)/meshes/${robot_name}/${motor_props['mesh']}" />
+            <mesh filename="package://andino_description/meshes/${robot_name}/${motor_props['mesh']}" />
           </xacro:if>
           <xacro:if value="${motor_props['scale'] != '' }" >
-            <mesh filename="file://$(find andino_description)/meshes/${robot_name}/${motor_props['mesh']}" scale="${motor_props['scale']}"/>
+            <mesh filename="package://andino_description/meshes/${robot_name}/${motor_props['mesh']}" scale="${motor_props['scale']}"/>
           </xacro:if>
         </geometry>
@@ -143,8 +143,8 @@
           <!-- The folder path get a folder_name global parameter -->
           <xacro:if value="${scale != '' }" >
-            <mesh filename="file://$(find andino_description)/meshes/${robot_name}/${mesh}" scale="${scale}"/>
+            <mesh filename="package://andino_description/meshes/${robot_name}/${mesh}" scale="${scale}"/>
           </xacro:if>
           <xacro:if value="${scale == '' }" >
-            <mesh filename="file://$(find andino_description)/meshes/${robot_name}/${mesh}" />
+            <mesh filename="package://andino_description/meshes/${robot_name}/${mesh}" />
           </xacro:if>
         </geometry>

Commit message: from file to package in the xacro
Signed-off-by: olmerg <olmerg@gmail.com>

File: andino_description/urdf/include/andino_caster_macro.urdf.xacro (robot description, xacro)
@@ -28,8 +28,8 @@
           <geometry>
             <xacro:if value="${scale != '' }" >
-              <mesh filename="file://$(find andino_description)/meshes/${robot_name}/${wheel_props['base']['mesh']}" scale="${scale}"/>
+              <mesh filename="package://andino_description/meshes/${robot_name}/${wheel_props['base']['mesh']}" scale="${scale}"/>
             </xacro:if>
             <xacro:if value="${scale == '' }" >
-              <mesh filename="file://$(find andino_description)/meshes/${robot_name}/${wheel_props['base']['mesh']}" />
+              <mesh filename="package://andino_description/meshes/${robot_name}/${wheel_props['base']['mesh']}" />
             </xacro:if>
           </geometry>
@@ -74,8 +74,8 @@
           <geometry>
             <xacro:if value="${scale != '' }" >
-              <mesh filename="file://$(find andino_description)/meshes/${robot_name}/${wheel_props['hub']['mesh']}" scale="${scale}"/>
+              <mesh filename="package://andino_description/meshes/${robot_name}/${wheel_props['hub']['mesh']}" scale="${scale}"/>
             </xacro:if>
             <xacro:if value="${scale == '' }" >
-              <mesh filename="file://$(find andino_description)/meshes/${robot_name}/${wheel_props['hub']['mesh']}" />
+              <mesh filename="package://andino_description/meshes/${robot_name}/${wheel_props['hub']['mesh']}" />
             </xacro:if>
           </geometry>
@@ -118,8 +118,8 @@
           <geometry>
             <xacro:if value="${scale != '' }" >
-              <mesh filename="file://$(find andino_description)/meshes/${robot_name}/${wheel_props['wheel']['mesh']}" scale="${scale}"/>
+              <mesh filename="package://andino_description/meshes/${robot_name}/${wheel_props['wheel']['mesh']}" scale="${scale}"/>
             </xacro:if>
             <xacro:if value="${scale == '' }" >
-              <mesh filename="file://$(find andino_description)/meshes/${robot_name}/${wheel_props['wheel']['mesh']}" />
+              <mesh filename="package://andino_description/meshes/${robot_name}/${wheel_props['wheel']['mesh']}" />
             </xacro:if>
           </geometry>

Commit message: Removes gazebo references from andino_description.
Signed-off-by: Franco Cipollone <franco.c@ekumenlabs.com>

File: andino_description/urdf/include/andino_caster_macro.urdf.xacro (robot description, xacro)
@@ -1,7 +1,9 @@
+<!--
+  Xacro macros were inspired on https://github.com/ros-mobile-robots/mobile_robot_description/wiki/
+-->
 <?xml version="1.0"?>
 <robot xmlns:xacro="http://www.ros.org/wiki/xacro">
 <!-- ===================== Caster xacro =========================================
-  Xacro to create caster links and the respective joints. For more detail information and usage, see:
-    https://github.com/pxalcantara/mobile_robot_description/wiki/Motor-xacro
+  Xacro to create caster links and the respective joints.
   params:
   - reflect [1/-1]: value to set the side of the caster;
@@ -12,8 +14,6 @@
 -->
 <!-- Caster wheel link & joint macro -->
-  <!-- locationprefix locationright wheel_base_dx TODO remove -->
   <xacro:macro name="caster_wheel"
                 params="reflect wheel_props locationright:=${0} scale:=''">
-    <!-- caster base (fixed) -->
     <link name="caster_base_link">
       <xacro:box_inertia  m="${wheel_props['base']['mass']}"
@@ -34,5 +34,4 @@
             </xacro:if>
           </geometry>
-          <!-- xacro:insert_block name="material_silver" / TODO use this block? -->
           <material name="silver"/>
         </visual>
@@ -62,7 +61,4 @@
       <dynamics damping="0.01" friction="0.0"/>
     </joint>
-    <gazebo reference="caster_base_link">
-      <material>Gazebo/Grey</material>
-    </gazebo>
     <!-- caster hub -->
     <link name="caster_rotation_link">
@@ -84,5 +80,4 @@
             </xacro:if>
           </geometry>
-          <!-- xacro:insert_block name="material_silver" / TODO use this block? -->
           <material name="silver"/>
         </visual>
@@ -112,7 +107,4 @@
       <dynamics damping="0.01" friction="0.0"/>
     </joint>
-    <gazebo reference="caster_rotation_link">
-      <material>Gazebo/Grey</material>
-    </gazebo>
     <!-- caster wheel -->
     <link name="caster_wheel_link">
@@ -120,5 +112,4 @@
                               r="${wheel_props['wheel']['radius']}"
                               l="${wheel_props['wheel']['length']}">
-        <!-- TODO unused block error?: origin xyz="0 0 0" rpy="${pi/2} 0 0" /-->
       </xacro:cylinder_inertia>
       <xacro:if value="${wheel_props['wheel']['mesh'] != '' }" >
@@ -133,5 +124,4 @@
             </xacro:if>
           </geometry>
-          <!-- TODO use this?: xacro:insert_block name="material_dark_grey" /-->
           <material name="black"/>
         </visual>
@@ -160,7 +150,4 @@
       <axis xyz="0 1 0" />
     </joint>
-    <gazebo reference="caster_wheel_link">
-      <material>Gazebo/DarkGrey</material>
-    </gazebo>
   </xacro:macro>
 </robot>

File: andino_description/urdf/include/common_macros.urdf.xacro (robot description, xacro)
@@ -54,7 +54,4 @@
       </xacro:cylinder_inertia>
     </link>
-    <gazebo reference="${prefix}_wheel">
-      <material>Gazebo/Grey</material>
-    </gazebo>
     <joint name="${prefix}_wheel_joint" type="continuous">
       <axis xyz="0 1 0" rpy="0 0 0" />

Commit message: caster_rotation fixed
Signed-off-by: olmerg <olmerg@gmail.com>

File: andino_description/urdf/include/andino_caster_macro.urdf.xacro (robot description, xacro)
@@ -111,5 +111,6 @@
     </xacro:if>
     <xacro:unless value="${use_fixed}">
-      <joint name="caster_rotation_joint" type="continuous">
+      <!--TODO(olmerg) initial solution problem with ros control  -->
+      <joint name="caster_rotation_joint" type="fixed">
         <origin xyz="${wheel_props['hub']['dx']} ${-wheel_props['hub']['dy'] * locationright} ${wheel_props['hub']['dz']}"
                 rpy="0 0 0" />

File: andino_gazebo/urdf/andino.gazebo.xacro (robot description, xacro)
@@ -15,5 +15,6 @@
   <xacro:friction reference="front_left_wheel" mu="100.0"/>
   <xacro:friction reference="caster_wheel_link" mu="0.05"/>
-  <xacro:friction reference="caster_rotation_link" mu="0.0"/>
+  <!--TODO(olmerg) initial solution problem with ros control  -->
+  <!-- <xacro:friction reference="caster_rotation_link" mu="0.0"/> -->
    <xacro:if value="$(arg use_gazebo_ros_control)">
     <ros2_control name="diff_controller" type="system">
@@ -49,5 +50,5 @@
       <update_rate>10</update_rate>
       <joint_name>caster_wheel_joint</joint_name>
-      <joint_name>caster_rotation_joint</joint_name>
+      <!-- <joint_name>caster_rotation_joint</joint_name> -->
     </plugin>
     </gazebo>
@@ -64,5 +65,5 @@
       <joint_name>left_wheel_joint</joint_name>
       <joint_name>caster_wheel_joint</joint_name>
-      <joint_name>caster_rotation_joint</joint_name>
+      <!-- <joint_name>caster_rotation_joint</joint_name> -->
     </plugin>
     <plugin name='andino_diff_drive' filename='libgazebo_ros_diff_drive.so'>

Commit message: moving the caster hack to spawn_launch
Signed-off-by: olmerg <olmerg@gmail.com>

File: andino_description/urdf/include/andino_caster_macro.urdf.xacro (robot description, xacro)
@@ -111,6 +111,5 @@
     </xacro:if>
     <xacro:unless value="${use_fixed}">
-      <!--TODO(olmerg) initial solution problem with ros control  -->
-      <joint name="caster_rotation_joint" type="fixed">
+      <joint name="caster_rotation_joint" type="continuous">
         <origin xyz="${wheel_props['hub']['dx']} ${-wheel_props['hub']['dy'] * locationright} ${wheel_props['hub']['dz']}"
                 rpy="0 0 0" />

File: andino_gazebo/urdf/andino.gazebo.xacro (robot description, xacro)
@@ -50,5 +50,4 @@
       <update_rate>10</update_rate>
       <joint_name>caster_wheel_joint</joint_name>
-      <!-- <joint_name>caster_rotation_joint</joint_name> -->
     </plugin>
     </gazebo>
@@ -65,5 +64,4 @@
       <joint_name>left_wheel_joint</joint_name>
       <joint_name>caster_wheel_joint</joint_name>
-      <!-- <joint_name>caster_rotation_joint</joint_name> -->
     </plugin>
     <plugin name='andino_diff_drive' filename='libgazebo_ros_diff_drive.so'>

Commit message: Update caster wheel colission mesh.
Signed-off-by: Miguel <miguel.diaz@creativa77.com.ar>

File: andino_description/urdf/include/andino_caster_macro.urdf.xacro (robot description, xacro)
@@ -45,7 +45,7 @@
       </xacro:if>
       <collision>
-        <origin xyz="0 0 ${-wheel_props['wheel']['size']['z']/2.0}" rpy="0 0 0" />
+        <origin xyz="0 0 ${-wheel_props['wheel']['radius']}" rpy="0 0 0" />
         <geometry>
-          <box size="${wheel_props['wheel']['size']['x']} ${wheel_props['wheel']['size']['y']} ${wheel_props['wheel']['size']['z']}" />
+          <sphere radius="${wheel_props['wheel']['radius']}" />
         </geometry>
       </collision>
