Commit message: Dev/migueldiaz/update andino chasis urdf (#296)
Update URDF and dependencies to use the new andino chasis. 

---------

Signed-off-by: Miguel <miguel.diaz@creativa77.com.ar>
Co-authored-by: Mmiguel Diaz <AngelDiaz03>
Co-authored-by: Miguel <miguel.diaz@creativa77.com.ar>

File: andino_description/urdf/include/andino_caster_macro.urdf.xacro (robot description, xacro)
@@ -5,8 +5,5 @@
 -->
 <!-- ===================== Caster xacro =========================================
-  Xacro to create caster links and the respective joints.
   params:
-  - reflect [1/-1]: value to set the side of the caster;
-  - use_fixed [bool]: wheter to use a fixed model or not
   - wheel_props [dictionary]: wheel properties;
   - base_props [dictionary]: base link properties;
@@ -16,117 +13,15 @@
 <!-- Caster wheel link & joint macro -->
   <xacro:macro name="caster_wheel"
-                params="reflect use_fixed wheel_props locationright:=${0} scale:=''">
-    <link name="caster_base_link">
-      <xacro:box_inertia  m="${wheel_props['base']['mass']}"
-                          x="${wheel_props['base']['size']['x']}"
-                          y="${wheel_props['base']['size']['y']}"
-                          z="${wheel_props['base']['size']['z']}"
-                          o_xyz="0.0 0.0 ${-wheel_props['base']['size']['z']/2.0}"
+                params="wheel_props scale:=''">
+    <link name="caster_link">
+      <xacro:box_inertia  m="${wheel_props['wheel']['mass']}"
+                          x="${wheel_props['wheel']['size']['x']}"
+                          y="${wheel_props['wheel']['size']['y']}"
+                          z="${wheel_props['wheel']['size']['z']}"
+                          o_xyz="0.0 0.0 ${-wheel_props['wheel']['size']['z']/2.0}"
                           o_rpy="0.0 0.0 0.0" />
-      <xacro:if value="${wheel_props['base']['mesh'] != '' }" >
-        <visual>
-          <origin xyz="0 0 ${-wheel_props['base']['size']['z']/2.0}" rpy="0 0 0" />
-          <geometry>
-            <xacro:if value="${scale != '' }" >
-              <mesh filename="package://andino_description/meshes/${robot_name}/${wheel_props['base']['mesh']}" scale="${scale}"/>
-            </xacro:if>
-            <xacro:if value="${scale == '' }" >
-              <mesh filename="package://andino_description/meshes/${robot_name}/${wheel_props['base']['mesh']}" />
-            </xacro:if>
-          </geometry>
-          <material name="silver"/>
-        </visual>
-      </xacro:if>
-      <xacro:if value="${wheel_props['base']['mesh'] == '' }" >
-        <visual>
-          <origin xyz="0 0 ${-wheel_props['base']['size']['z']/2.0}" rpy="0 0 0" />
-          <geometry>
-            <box size="${wheel_props['base']['size']['x']} ${wheel_props['base']['size']['y']} ${wheel_props['base']['size']['z']}" />
-          </geometry>
-          <material name="red"/>
-        </visual>
-      </xacro:if>
-      <collision>
-        <origin xyz="0 0 ${-wheel_props['base']['size']['z']/2.0}" rpy="0 0 0" />
-        <geometry>
-          <box size="${wheel_props['base']['size']['x']} ${wheel_props['base']['size']['y']} ${wheel_props['base']['size']['z']}" />
-        </geometry>
-      </collision>
-    </link>
-    <joint name="caster_base_joint" type="fixed">
-      <origin xyz="${wheel_props['base']['dx']} ${-wheel_props['base']['dy'] * locationright} ${wheel_props['base']['dz']}"
-              rpy="0 0 0" />
-      <parent link="base_link" />
-      <child link="caster_base_link" />
-      <axis xyz="0 0 1" />
-      <dynamics damping="0.01" friction="0.0"/>
-    </joint>
-    <!-- caster hub -->
-    <link name="caster_rotation_link">
-      <xacro:box_inertia  m="${wheel_props['hub']['mass']}"
-                          x="${wheel_props['hub']['size']['x']}"
-                          y="${wheel_props['hub']['size']['y']}"
-                          z="${wheel_props['hub']['size']['z']}"
-                          o_xyz="0.0 0.0 ${-wheel_props['hub']['size']['z']/2.0}"
-                          o_rpy="0.0 0.0 0.0" />
-      <xacro:if value="${wheel_props['hub']['mesh'] != '' }" >
-        <visual>
-          <origin xyz="0 0 ${-wheel_props['hub']['size']['z']/2.0}" rpy="0 0 0" />
-          <geometry>
-            <xacro:if value="${scale != '' }" >
-              <mesh filename="package://andino_description/meshes/${robot_name}/${wheel_props['hub']['mesh']}" scale="${scale}"/>
-            </xacro:if>
-            <xacro:if value="${scale == '' }" >
-              <mesh filename="package://andino_description/meshes/${robot_name}/${wheel_props['hub']['mesh']}" />
-            </xacro:if>
-          </geometry>
-          <material name="silver"/>
-        </visual>
-      </xacro:if>
-      <xacro:if value="${wheel_props['hub']['mesh'] == '' }" >
-        <visual>
-          <origin xyz="0 0 ${-wheel_props['hub']['size']['z']/2.0}" rpy="0 0 0" />
-          <geometry>
-            <box size="${wheel_props['hub']['size']['x']} ${wheel_props['hub']['size']['y']} ${wheel_props['hub']['size']['z']}" />
-          </geometry>
-          <material name="red"/>
-        </visual>
-      </xacro:if>
-      <collision>
-        <origin xyz="0 0 ${-wheel_props['hub']['size']['z']/2.0}" rpy="0 0 0" />
-        <geometry>
-          <box size="${wheel_props['hub']['size']['x']} ${wheel_props['hub']['size']['y']} ${wheel_props['hub']['size']['z']}" />
-        </geometry>
-      </collision>
-    </link>
-    <xacro:if value="${use_fixed}">
-      <joint name="caster_rotation_joint" type="fixed">
-        <origin xyz="${wheel_props['hub']['dx']} ${-wheel_props['hub']['dy'] * locationright} ${wheel_props['hub']['dz']}"
-                rpy="0 0 0" />
-        <parent link="base_link" />
-        <child link="caster_rotation_link" />
-        <axis xyz="0 0 1" />
-        <dynamics damping="0.01" friction="0.0"/>
-      </joint>
-    </xacro:if>
-    <xacro:unless value="${use_fixed}">
-      <joint name="caster_rotation_joint" type="continuous">
-        <origin xyz="${wheel_props['hub']['dx']} ${-wheel_props['hub']['dy'] * locationright} ${wheel_props['hub']['dz']}"
-                rpy="0 0 0" />
-        <parent link="base_link" />
-        <child link="caster_rotation_link" />
-        <axis xyz="0 0 1" />
-        <dynamics damping="0.01" friction="0.0"/>
-      </joint>
-    </xacro:unless>
-    <!-- caster wheel -->
-    <link name="caster_wheel_link">
-      <xacro:cylinder_inertia m="${wheel_props['wheel']['mass']}"
-                              r="${wheel_props['wheel']['radius']}"
-                              l="${wheel_props['wheel']['length']}">
-      </xacro:cylinder_inertia>
       <xacro:if value="${wheel_props['wheel']['mesh'] != '' }" >
         <visual>
-          <origin xyz="0 0 0" rpy="0 0 0" />
+          <origin xyz="0 0 0" rpy="${pi} 0 ${pi/2}" />
           <geometry>
             <xacro:if value="${scale != '' }" >
@@ -137,12 +32,12 @@
             </xacro:if>
           </geometry>
-          <material name="black"/>
+          <material name="silver"/>
         </visual>
       </xacro:if>
       <xacro:if value="${wheel_props['wheel']['mesh'] == '' }" >
         <visual>
-          <origin xyz="0 0 0" rpy="${pi/2} 0 0" />
+          <origin xyz="0 0 ${-wheel_props['wheel']['size']['z']/2.0}" rpy="0 0 0" />
           <geometry>
-            <cylinder length="${wheel_props['wheel']['length']}" radius="${wheel_props['wheel']['radius']}" />
+            <box size="${wheel_props['wheel']['size']['x']} ${wheel_props['wheel']['size']['y']} ${wheel_props['wheel']['size']['z']}" />
           </geometry>
           <material name="red"/>
@@ -150,28 +45,18 @@
       </xacro:if>
       <collision>
-        <origin xyz="0 0 0" rpy="${pi/2} 0 0" />
+        <origin xyz="0 0 ${-wheel_props['wheel']['radius']}" rpy="0 0 0" />
         <geometry>
-          <cylinder length="${wheel_props['wheel']['length']}" radius="${wheel_props['wheel']['radius']}" />
+          <sphere radius="${wheel_props['wheel']['radius']}" />
         </geometry>
       </collision>
     </link>
-    <xacro:if value="${use_fixed}">
-      <joint name="caster_wheel_joint" type="fixed">
-        <origin xyz="${wheel_props['wheel']['dx']} ${-wheel_props['wheel']['dy'] * locationright} ${wheel_props['wheel']['dz']}"
-                rpy="0 0 0" />
-        <parent link="caster_rotation_link" />
-        <child link="caster_wheel_link" />
-        <axis xyz="0 1 0" />
-      </joint>
-    </xacro:if>
-    <xacro:unless value="${use_fixed}">
-      <joint name="caster_wheel_joint" type="continuous">
-        <origin xyz="${wheel_props['wheel']['dx']} ${-wheel_props['wheel']['dy'] * locationright} ${wheel_props['wheel']['dz']}"
-                rpy="0 0 0" />
-        <parent link="caster_rotation_link" />
-        <child link="caster_wheel_link" />
-        <axis xyz="0 1 0" />
-      </joint>
-    </xacro:unless>
+    <joint name="caster_base_joint" type="fixed">
+      <origin xyz="${wheel_props['wheel']['dx']} ${wheel_props['wheel']['dy']} ${wheel_props['wheel']['dz']}"
+              rpy="0 0 0" />
+      <parent link="base_link" />
+      <child link="caster_link" />
+      <axis xyz="0 0 1" />
+      <dynamics damping="0.01" friction="0.0"/>
+    </joint>
   </xacro:macro>
 </robot>
