Commit message: gz_classic_sim: Free caster wheel joint.
Signed-off-by: Franco Cipollone <franco.c@ekumenlabs.com>

File: andino_gz_classic/urdf/andino_gz_classic.xacro (robot description, xacro)
@@ -2,19 +2,4 @@
 <robot xmlns:xacro="http://www.ros.org/wiki/xacro" name="andino">
   <xacro:include filename="$(find andino_description)/urdf/andino.urdf.xacro"/>
-  <xacro:macro name="friction" params="reference mu">
-    <gazebo reference="${reference}">
-      <mu1>${mu}</mu1>
-      <mu2>${mu}</mu2>
-      <kp>1000000.0</kp>
-      <kd>1.0</kd>
-      <minDepth>0.0001</minDepth>
-      <maxVel>1.0</maxVel>
-    </gazebo>
-  </xacro:macro>
-  <xacro:friction reference="right_wheel" mu="100.0"/>
-  <xacro:friction reference="left_wheel" mu="100.0"/>
-  <xacro:friction reference="caster_wheel_link" mu="0.05"/>
-  <!--TODO(olmerg) initial solution problem with ros control  -->
-  <!-- <xacro:friction reference="caster_rotation_link" mu="0.0"/> -->
    <xacro:if value="$(arg use_gazebo_ros_control)">
     <ros2_control name="diff_controller" type="system">
@@ -48,5 +33,6 @@
         <remapping>/tf:=tf</remapping>
       </ros>
-      <update_rate>10</update_rate>
+      <update_rate>30</update_rate>
+      <joint_name>caster_rotation_joint</joint_name>
       <joint_name>caster_wheel_joint</joint_name>
     </plugin>
@@ -60,7 +46,8 @@
         <remapping>/tf:=tf</remapping>
       </ros>
-      <update_rate>10</update_rate>
+      <update_rate>30</update_rate>
       <joint_name>right_wheel_joint</joint_name>
       <joint_name>left_wheel_joint</joint_name>
+      <joint_name>caster_rotation_joint</joint_name>
       <joint_name>caster_wheel_joint</joint_name>
     </plugin>
