Commit message: Renames andino_description package.
Signed-off-by: Franco Cipollone <franco.c@ekumenlabs.com>

File: andino_description/urdf/andino.urdf.xacro (robot description, xacro)
@@ -1,9 +1,9 @@
 <?xml version="1.0"?>
-<robot xmlns:xacro="http://www.ros.org/wiki/xacro" name="carpincho">
-  <xacro:property name="package_name" value="carpincho_description"/>
-  <xacro:property name="robot_name" value="carpincho"/>
+<robot xmlns:xacro="http://www.ros.org/wiki/xacro" name="andino">
+  <xacro:property name="package_name" value="andino_description"/>
+  <xacro:property name="robot_name" value="andino"/>
   <xacro:include filename="$(find ${package_name})/urdf/include/common_macros.urdf.xacro" />
   <xacro:include filename="$(find ${package_name})/urdf/include/common_sensors.urdf.xacro" />
-  <xacro:include filename="$(find ${package_name})/urdf/include/carpincho_caster_macro.urdf.xacro" />
+  <xacro:include filename="$(find ${package_name})/urdf/include/andino_caster_macro.urdf.xacro" />
   <xacro:property name="caster_wheel_yaml" value="$(find ${package_name})/config/${robot_name}/caster_wheel.yaml" />
   <xacro:property name="caster_wheel_props" value="${xacro.load_yaml(caster_wheel_yaml)}"/>
@@ -61,4 +61,4 @@
   </xacro:camera_sensor>
   <!-- ros2_control -->
-  <xacro:include filename="$(find ${package_name})/urdf/include/carpincho_control.urdf.xacro" />
+  <xacro:include filename="$(find ${package_name})/urdf/include/andino_control.urdf.xacro" />
 </robot>

File: andino_description/urdf/include/andino_caster_macro.urdf.xacro (robot description, xacro)
@@ -28,8 +28,8 @@
           <geometry>
             <xacro:if value="${scale != '' }" >
-              <mesh filename="package://carpincho_description/meshes/${robot_name}/${wheel_props['base']['mesh']}" scale="${scale}"/>
+              <mesh filename="package://andino_description/meshes/${robot_name}/${wheel_props['base']['mesh']}" scale="${scale}"/>
             </xacro:if>
             <xacro:if value="${scale == '' }" >
-              <mesh filename="package://carpincho_description/meshes/${robot_name}/${wheel_props['base']['mesh']}" />
+              <mesh filename="package://andino_description/meshes/${robot_name}/${wheel_props['base']['mesh']}" />
             </xacro:if>
           </geometry>
@@ -78,8 +78,8 @@
           <geometry>
             <xacro:if value="${scale != '' }" >
-              <mesh filename="package://carpincho_description/meshes/${robot_name}/${wheel_props['hub']['mesh']}" scale="${scale}"/>
+              <mesh filename="package://andino_description/meshes/${robot_name}/${wheel_props['hub']['mesh']}" scale="${scale}"/>
             </xacro:if>
             <xacro:if value="${scale == '' }" >
-              <mesh filename="package://carpincho_description/meshes/${robot_name}/${wheel_props['hub']['mesh']}" />
+              <mesh filename="package://andino_description/meshes/${robot_name}/${wheel_props['hub']['mesh']}" />
             </xacro:if>
           </geometry>
@@ -127,8 +127,8 @@
           <geometry>
             <xacro:if value="${scale != '' }" >
-              <mesh filename="package://carpincho_description/meshes/${robot_name}/${wheel_props['wheel']['mesh']}" scale="${scale}"/>
+              <mesh filename="package://andino_description/meshes/${robot_name}/${wheel_props['wheel']['mesh']}" scale="${scale}"/>
             </xacro:if>
             <xacro:if value="${scale == '' }" >
-              <mesh filename="package://carpincho_description/meshes/${robot_name}/${wheel_props['wheel']['mesh']}" />
+              <mesh filename="package://andino_description/meshes/${robot_name}/${wheel_props['wheel']['mesh']}" />
             </xacro:if>
           </geometry>

File: andino_description/urdf/include/andino_control.urdf.xacro (robot description, xacro)
@@ -1,8 +1,8 @@
 <?xml version="1.0"?>
 <robot xmlns:xacro="http://www.ros.org/wiki/xacro">
-  <!-- TODO(francocipollone): This xacro should be part of carpincho_control package instead.-->
+  <!-- TODO(francocipollone): This xacro should be part of andino_control package instead.-->
   <ros2_control name="RealRobot" type="system">
     <hardware>
-      <plugin>carpincho_base/DiffDriveCarpincho</plugin>
+      <plugin>andino_base/DiffDriveAndino</plugin>
       <!-- TODO(francocipollone): Parameters like loop_rate, device, baud_rate, etc should be loaded from a file or passed via the launch file as xacro args -->
       <param name="left_wheel_name">left_wheel_joint</param>

File: andino_description/urdf/include/common_macros.urdf.xacro (robot description, xacro)
@@ -23,8 +23,8 @@
         <geometry>
           <xacro:if value="${wheel_props['scale'] == '' }" >
-            <mesh filename="package://carpincho_description/meshes/${robot_name}/${wheel_props['mesh']}" />
+            <mesh filename="package://andino_description/meshes/${robot_name}/${wheel_props['mesh']}" />
           </xacro:if>
           <xacro:if value="${wheel_props['scale'] == '' }" >
-            <mesh filename="package://carpincho_description/meshes/${robot_name}/${wheel_props['mesh']}" scale="${wheel_props['scale']}" />
+            <mesh filename="package://andino_description/meshes/${robot_name}/${wheel_props['mesh']}" scale="${wheel_props['scale']}" />
           </xacro:if>
         </geometry>
@@ -87,8 +87,8 @@
         <geometry>
           <xacro:if value="${motor_props['scale'] == '' }" >
-            <mesh filename="package://carpincho_description/meshes/${robot_name}/${motor_props['mesh']}" />
+            <mesh filename="package://andino_description/meshes/${robot_name}/${motor_props['mesh']}" />
           </xacro:if>
           <xacro:if value="${motor_props['scale'] != '' }" >
-            <mesh filename="package://carpincho_description/meshes/${robot_name}/${motor_props['mesh']}" scale="${motor_props['scale']}"/>
+            <mesh filename="package://andino_description/meshes/${robot_name}/${motor_props['mesh']}" scale="${motor_props['scale']}"/>
           </xacro:if>
         </geometry>
@@ -146,8 +146,8 @@
           <!-- The folder path get a folder_name global parameter -->
           <xacro:if value="${scale != '' }" >
-            <mesh filename="package://carpincho_description/meshes/${robot_name}/${mesh}" scale="${scale}"/>
+            <mesh filename="package://andino_description/meshes/${robot_name}/${mesh}" scale="${scale}"/>
           </xacro:if>
           <xacro:if value="${scale == '' }" >
-            <mesh filename="package://carpincho_description/meshes/${robot_name}/${mesh}" />
+            <mesh filename="package://andino_description/meshes/${robot_name}/${mesh}" />
           </xacro:if>
         </geometry>

File: andino_description/urdf/include/common_sensors.urdf.xacro (robot description, xacro)
@@ -9,5 +9,5 @@
       <origin xyz="0 0 0" rpy="0 0 ${pi}"/>
       <geometry>
-        <mesh filename="package://carpincho_description/meshes/sensors/${mesh}" />
+        <mesh filename="package://andino_description/meshes/sensors/${mesh}" />
       </geometry>
       <material name="dark_grey"/>

Commit message: Adds camera mount mesh and adjusts sizes.
Signed-off-by: Franco Cipollone <franco.c@ekumenlabs.com>

File: andino_description/urdf/andino.urdf.xacro (robot description, xacro)
@@ -24,5 +24,5 @@
   <!-- Second story link -->
   <xacro:base link_name="second_base_link" base_prop="${base_props}" mesh="${base_props['base']['mesh']}" >
-    <origin xyz="0 0 0.03" rpy="0 0 0" />
+    <origin xyz="0 0 0.05" rpy="0 0 0" />
   </xacro:base>
   <!-- Joint to connect second_story with base_link -->

Commit message: Add optional parameter to generate Fixed/Coninuous caster joint
Signed-off-by: Christian Barcelo <christianbarcelo@ekumenlabs.com>

File: andino_description/urdf/andino.urdf.xacro (robot description, xacro)
@@ -8,4 +8,5 @@
   <xacro:property name="caster_wheel_yaml" value="$(find ${package_name})/config/${robot_name}/caster_wheel.yaml" />
   <xacro:property name="caster_wheel_props" value="${xacro.load_yaml(caster_wheel_yaml)}"/>
+  <xacro:arg name="use_fixed_caster" default="True"/>
   <xacro:property name="wheel_yaml" value="$(find ${package_name})/config/${robot_name}/wheel.yaml" />
   <xacro:property name="wheel_props" value="${xacro.load_yaml(wheel_yaml)}"/>
@@ -34,4 +35,5 @@
   <!-- Caster Wheel -->
   <xacro:caster_wheel reflect="-1"
+                      use_fixed="$(arg use_fixed_caster)"
                       wheel_props="${caster_wheel_props}">
   </xacro:caster_wheel>

File: andino_description/urdf/include/andino_caster_macro.urdf.xacro (robot description, xacro)
@@ -8,4 +8,5 @@
   params:
   - reflect [1/-1]: value to set the side of the caster;
+  - use_fixed [bool]: wheter to use a fixed model or not
   - wheel_props [dictionary]: wheel properties;
   - base_props [dictionary]: base link properties;
@@ -15,5 +16,5 @@
 <!-- Caster wheel link & joint macro -->
   <xacro:macro name="caster_wheel"
-                params="reflect wheel_props locationright:=${0} scale:=''">
+                params="reflect use_fixed wheel_props locationright:=${0} scale:=''">
     <link name="caster_base_link">
       <xacro:box_inertia  m="${wheel_props['base']['mass']}"
@@ -99,12 +100,24 @@
       </collision>
     </link>
-    <joint name="caster_rotation_joint" type="fixed">
-      <origin xyz="${wheel_props['hub']['dx']} ${-wheel_props['hub']['dy'] * locationright} ${wheel_props['hub']['dz']}"
-              rpy="0 0 0" />
-      <parent link="base_link" />
-      <child link="caster_rotation_link" />
-      <axis xyz="0 0 1" />
-      <dynamics damping="0.01" friction="0.0"/>
-    </joint>
+    <xacro:if value="${use_fixed}">
+      <joint name="caster_rotation_joint" type="fixed">
+        <origin xyz="${wheel_props['hub']['dx']} ${-wheel_props['hub']['dy'] * locationright} ${wheel_props['hub']['dz']}"
+                rpy="0 0 0" />
+        <parent link="base_link" />
+        <child link="caster_rotation_link" />
+        <axis xyz="0 0 1" />
+        <dynamics damping="0.01" friction="0.0"/>
+      </joint>
+    </xacro:if>
+    <xacro:unless value="${use_fixed}">
+      <joint name="caster_rotation_joint" type="continuous">
+        <origin xyz="${wheel_props['hub']['dx']} ${-wheel_props['hub']['dy'] * locationright} ${wheel_props['hub']['dz']}"
+                rpy="0 0 0" />
+        <parent link="base_link" />
+        <child link="caster_rotation_link" />
+        <axis xyz="0 0 1" />
+        <dynamics damping="0.01" friction="0.0"/>
+      </joint>
+    </xacro:unless>
     <!-- caster wheel -->
     <link name="caster_wheel_link">
@@ -143,11 +156,22 @@
       </collision>
     </link>
-    <joint name="caster_wheel_joint" type="fixed">
-      <origin xyz="${wheel_props['wheel']['dx']} ${-wheel_props['wheel']['dy'] * locationright} ${wheel_props['wheel']['dz']}"
-              rpy="0 0 0" />
-      <parent link="caster_rotation_link" />
-      <child link="caster_wheel_link" />
-      <axis xyz="0 1 0" />
-    </joint>
+    <xacro:if value="${use_fixed}">
+      <joint name="caster_wheel_joint" type="fixed">
+        <origin xyz="${wheel_props['wheel']['dx']} ${-wheel_props['wheel']['dy'] * locationright} ${wheel_props['wheel']['dz']}"
+                rpy="0 0 0" />
+        <parent link="caster_rotation_link" />
+        <child link="caster_wheel_link" />
+        <axis xyz="0 1 0" />
+      </joint>
+    </xacro:if>
+    <xacro:unless value="${use_fixed}">
+      <joint name="caster_wheel_joint" type="continuous">
+        <origin xyz="${wheel_props['wheel']['dx']} ${-wheel_props['wheel']['dy'] * locationright} ${wheel_props['wheel']['dz']}"
+                rpy="0 0 0" />
+        <parent link="caster_rotation_link" />
+        <child link="caster_wheel_link" />
+        <axis xyz="0 1 0" />
+      </joint>
+    </xacro:unless>
   </xacro:macro>
 </robot>

Commit message: caster in gazebo/ros_control with drift
Signed-off-by: olmerg <olmerg@gmail.com>

File: andino_description/urdf/andino.urdf.xacro (robot description, xacro)
@@ -9,4 +9,5 @@
   <xacro:property name="caster_wheel_props" value="${xacro.load_yaml(caster_wheel_yaml)}"/>
   <xacro:arg name="use_fixed_caster" default="True"/>
+  <xacro:arg name="use_real_ros_control" default="True"/>
   <xacro:property name="wheel_yaml" value="$(find ${package_name})/config/${robot_name}/wheel.yaml" />
   <xacro:property name="wheel_props" value="${xacro.load_yaml(wheel_yaml)}"/>
@@ -63,4 +64,6 @@
   </xacro:camera_sensor>
   <!-- ros2_control -->
+  <xacro:if value="$(arg use_real_ros_control)">
   <xacro:include filename="$(find ${package_name})/urdf/include/andino_control.urdf.xacro" />
+  </xacro:if>
 </robot>

File: andino_description/urdf/include/common_macros.urdf.xacro (robot description, xacro)
@@ -59,5 +59,5 @@
       <child link="${prefix}_wheel"/>
       <origin xyz="${pos_x_joint} ${reflect* pos_y_joint} ${pos_z_joint}" rpy="0 0 0"/>
-      <dynamics damping="0.0" friction="4.5"/>
+      <dynamics damping="0.01" friction="0.0"/>
     </joint>
   </xacro:macro>

File: andino_gazebo/urdf/andino.gazebo.xacro (robot description, xacro)
@@ -12,7 +12,8 @@
     </gazebo>
   </xacro:macro>
-  <xacro:friction reference="front_right_wheel" mu="10"/>
-  <xacro:friction reference="front_left_wheel" mu="10"/>
-  <xacro:friction reference="caster_wheel_link" mu="0.0"/>
+  <xacro:friction reference="front_right_wheel" mu="100.0"/>
+  <xacro:friction reference="front_left_wheel" mu="100.0"/>
+  <xacro:friction reference="caster_wheel_link" mu="0.05"/>
+  <xacro:friction reference="caster_rotation_link" mu="0.0"/>
    <xacro:if value="$(arg use_gazebo_ros_control)">
     <ros2_control name="diff_controller" type="system">
@@ -41,4 +42,13 @@
           <parameters>$(find andino_control)/config/andino_controllers.yaml</parameters>
       </plugin>
+      <plugin name="andino_joint_state_caster" filename="libgazebo_ros_joint_state_publisher.so">
+      <ros>
+        <remapping>~/out:=joint_states</remapping>
+        <remapping>/tf:=tf</remapping>
+      </ros>
+      <update_rate>10</update_rate>
+      <joint_name>caster_wheel_joint</joint_name>
+      <joint_name>caster_rotation_joint</joint_name>
+    </plugin>
     </gazebo>
   </xacro:if>
@@ -53,4 +63,6 @@
       <joint_name>right_wheel_joint</joint_name>
       <joint_name>left_wheel_joint</joint_name>
+      <joint_name>caster_wheel_joint</joint_name>
+      <joint_name>caster_rotation_joint</joint_name>
     </plugin>
     <plugin name='andino_diff_drive' filename='libgazebo_ros_diff_drive.so'>
@@ -60,6 +72,6 @@
       </ros>
       <!-- wheels -->
-      <left_joint>right_wheel_joint</left_joint>
-      <right_joint>left_wheel_joint</right_joint>
+      <left_joint>left_wheel_joint</left_joint>
+      <right_joint>right_wheel_joint</right_joint>
       <!-- kinematics -->
       <wheel_separation>0.137</wheel_separation>

Commit message: Parametrize config yaml path in andino.urdf.xacro

File: andino_description/urdf/andino.urdf.xacro (robot description, xacro)
@@ -6,15 +6,16 @@
   <xacro:include filename="$(find ${package_name})/urdf/include/common_sensors.urdf.xacro" />
   <xacro:include filename="$(find ${package_name})/urdf/include/andino_caster_macro.urdf.xacro" />
-  <xacro:property name="caster_wheel_yaml" value="$(find ${package_name})/config/${robot_name}/caster_wheel.yaml" />
+  <xacro:arg name="config_yaml_path" default="$(find ${package_name})/config/${robot_name}" />
+  <xacro:property name="caster_wheel_yaml" value="$(arg config_yaml_path)/caster_wheel.yaml" />
   <xacro:property name="caster_wheel_props" value="${xacro.load_yaml(caster_wheel_yaml)}"/>
   <xacro:arg name="use_fixed_caster" default="True"/>
   <xacro:arg name="use_real_ros_control" default="True"/>
-  <xacro:property name="wheel_yaml" value="$(find ${package_name})/config/${robot_name}/wheel.yaml" />
+  <xacro:property name="wheel_yaml" value="$(arg config_yaml_path)/wheel.yaml" />
   <xacro:property name="wheel_props" value="${xacro.load_yaml(wheel_yaml)}"/>
-  <xacro:property name="motor_yaml" value="$(find ${package_name})/config/${robot_name}/motor.yaml" />
+  <xacro:property name="motor_yaml" value="$(arg config_yaml_path)/motor.yaml" />
   <xacro:property name="motor_props" value="${xacro.load_yaml(motor_yaml)}"/>
-  <xacro:property name="base_yaml" value="$(find ${package_name})/config/${robot_name}/base.yaml" />
+  <xacro:property name="base_yaml" value="$(arg config_yaml_path)/base.yaml" />
   <xacro:property name="base_props" value="${xacro.load_yaml(base_yaml)}"/>
-  <xacro:property name="sensor_yaml" value="$(find ${package_name})/config/${robot_name}/sensors.yaml" />
+  <xacro:property name="sensor_yaml" value="$(arg config_yaml_path)/sensors.yaml" />
   <xacro:property name="sensor_prop" value="${xacro.load_yaml(sensor_yaml)}"/>
   <!-- Footprint link -->

Commit message: Rename arg to yaml_config_dir

File: andino_description/urdf/andino.urdf.xacro (robot description, xacro)
@@ -6,16 +6,16 @@
   <xacro:include filename="$(find ${package_name})/urdf/include/common_sensors.urdf.xacro" />
   <xacro:include filename="$(find ${package_name})/urdf/include/andino_caster_macro.urdf.xacro" />
-  <xacro:arg name="config_yaml_path" default="$(find ${package_name})/config/${robot_name}" />
-  <xacro:property name="caster_wheel_yaml" value="$(arg config_yaml_path)/caster_wheel.yaml" />
+  <xacro:arg name="yaml_config_dir" default="$(find ${package_name})/config/${robot_name}" />
+  <xacro:property name="caster_wheel_yaml" value="$(arg yaml_config_dir)/caster_wheel.yaml" />
   <xacro:property name="caster_wheel_props" value="${xacro.load_yaml(caster_wheel_yaml)}"/>
   <xacro:arg name="use_fixed_caster" default="True"/>
   <xacro:arg name="use_real_ros_control" default="True"/>
-  <xacro:property name="wheel_yaml" value="$(arg config_yaml_path)/wheel.yaml" />
+  <xacro:property name="wheel_yaml" value="$(arg yaml_config_dir)/wheel.yaml" />
   <xacro:property name="wheel_props" value="${xacro.load_yaml(wheel_yaml)}"/>
-  <xacro:property name="motor_yaml" value="$(arg config_yaml_path)/motor.yaml" />
+  <xacro:property name="motor_yaml" value="$(arg yaml_config_dir)/motor.yaml" />
   <xacro:property name="motor_props" value="${xacro.load_yaml(motor_yaml)}"/>
-  <xacro:property name="base_yaml" value="$(arg config_yaml_path)/base.yaml" />
+  <xacro:property name="base_yaml" value="$(arg yaml_config_dir)/base.yaml" />
   <xacro:property name="base_props" value="${xacro.load_yaml(base_yaml)}"/>
-  <xacro:property name="sensor_yaml" value="$(arg config_yaml_path)/sensors.yaml" />
+  <xacro:property name="sensor_yaml" value="$(arg yaml_config_dir)/sensors.yaml" />
   <xacro:property name="sensor_prop" value="${xacro.load_yaml(sensor_yaml)}"/>
   <!-- Footprint link -->

Commit message: Parametrizes config yaml path in andino.urdf.xacro (#137)

File: andino_description/urdf/andino.urdf.xacro (robot description, xacro)
@@ -6,15 +6,16 @@
   <xacro:include filename="$(find ${package_name})/urdf/include/common_sensors.urdf.xacro" />
   <xacro:include filename="$(find ${package_name})/urdf/include/andino_caster_macro.urdf.xacro" />
-  <xacro:property name="caster_wheel_yaml" value="$(find ${package_name})/config/${robot_name}/caster_wheel.yaml" />
+  <xacro:arg name="yaml_config_dir" default="$(find ${package_name})/config/${robot_name}" />
+  <xacro:property name="caster_wheel_yaml" value="$(arg yaml_config_dir)/caster_wheel.yaml" />
   <xacro:property name="caster_wheel_props" value="${xacro.load_yaml(caster_wheel_yaml)}"/>
   <xacro:arg name="use_fixed_caster" default="True"/>
   <xacro:arg name="use_real_ros_control" default="True"/>
-  <xacro:property name="wheel_yaml" value="$(find ${package_name})/config/${robot_name}/wheel.yaml" />
+  <xacro:property name="wheel_yaml" value="$(arg yaml_config_dir)/wheel.yaml" />
   <xacro:property name="wheel_props" value="${xacro.load_yaml(wheel_yaml)}"/>
-  <xacro:property name="motor_yaml" value="$(find ${package_name})/config/${robot_name}/motor.yaml" />
+  <xacro:property name="motor_yaml" value="$(arg yaml_config_dir)/motor.yaml" />
   <xacro:property name="motor_props" value="${xacro.load_yaml(motor_yaml)}"/>
-  <xacro:property name="base_yaml" value="$(find ${package_name})/config/${robot_name}/base.yaml" />
+  <xacro:property name="base_yaml" value="$(arg yaml_config_dir)/base.yaml" />
   <xacro:property name="base_props" value="${xacro.load_yaml(base_yaml)}"/>
-  <xacro:property name="sensor_yaml" value="$(find ${package_name})/config/${robot_name}/sensors.yaml" />
+  <xacro:property name="sensor_yaml" value="$(arg yaml_config_dir)/sensors.yaml" />
   <xacro:property name="sensor_prop" value="${xacro.load_yaml(sensor_yaml)}"/>
   <!-- Footprint link -->

Commit message: Add new mesh for second base
Signed-off-by: lneumarkt <leonardoneumarkt@ekumenlabs.com>

File: andino_description/urdf/andino.urdf.xacro (robot description, xacro)
@@ -17,4 +17,6 @@
   <xacro:property name="base_yaml" value="$(arg yaml_config_dir)/base.yaml" />
   <xacro:property name="base_props" value="${xacro.load_yaml(base_yaml)}"/>
+  <xacro:property name="second_base_yaml" value="$(arg yaml_config_dir)/second_base.yaml" />
+  <xacro:property name="second_base_props" value="${xacro.load_yaml(second_base_yaml)}"/>
   <xacro:property name="sensor_yaml" value="$(arg yaml_config_dir)/sensors.yaml" />
   <xacro:property name="sensor_prop" value="${xacro.load_yaml(sensor_yaml)}"/>
@@ -26,5 +28,5 @@
   </xacro:base>
   <!-- Second story link -->
-  <xacro:base link_name="second_base_link" base_prop="${base_props}" mesh="${base_props['base']['mesh']}" >
+  <xacro:base link_name="second_base_link" base_prop="${second_base_props}" mesh="${second_base_props['base']['mesh']}" >
     <origin xyz="0 0 0.05" rpy="0 0 0" />
   </xacro:base>
