Commit message: Update caster wheel.
Signed-off-by: Miguel <miguel.diaz@creativa77.com.ar>

File: andino_description/urdf/andino.urdf.xacro (robot description, xacro)
@@ -17,6 +17,8 @@
   <xacro:property name="base_yaml" value="$(arg yaml_config_dir)/base.yaml" />
   <xacro:property name="base_props" value="${xacro.load_yaml(base_yaml)}"/>
-  <xacro:property name="second_base_yaml" value="$(arg yaml_config_dir)/second_base.yaml" />
-  <xacro:property name="second_base_props" value="${xacro.load_yaml(second_base_yaml)}"/>
+  <xacro:property name="lidar_base_yaml" value="$(arg yaml_config_dir)/lidar_base.yaml" />
+  <xacro:property name="lidar_base_props" value="${xacro.load_yaml(lidar_base_yaml)}"/>
+  <xacro:property name="battery_base_yaml" value="$(arg yaml_config_dir)/battery_base.yaml" />
+  <xacro:property name="battery_base_props" value="${xacro.load_yaml(battery_base_yaml)}"/>
   <xacro:property name="sensor_yaml" value="$(arg yaml_config_dir)/sensors.yaml" />
   <xacro:property name="sensor_prop" value="${xacro.load_yaml(sensor_yaml)}"/>
@@ -27,29 +29,37 @@
   <!-- Base link -->
   <xacro:base link_name="base_link" base_prop="${base_props}" mesh="${base_props['base']['mesh']}" >
-    <origin xyz="0 0 0" rpy="0 0 0" />
+    <origin xyz="0 0 0" rpy="0 0 ${pi}" />
   </xacro:base>
-  <!-- Second story link -->
-  <xacro:base link_name="second_base_link" base_prop="${second_base_props}" mesh="${second_base_props['base']['mesh']}" >
-    <origin xyz="0 0 0.05" rpy="0 0 0" />
+  <!-- Lidar base link -->
+  <xacro:base link_name="lidar_base_link" base_prop="${lidar_base_props}" mesh="${lidar_base_props['base']['mesh']}" >
+    <origin xyz="0.062067 0 0.08" rpy="0 ${pi} 0" />
   </xacro:base>
   <!-- Joint to connect second_story with base_link -->
-  <joint name="second_base_joint" type="fixed">
+  <joint name="lidar_base_joint" type="fixed">
     <parent link="base_link"/>
-    <child link="second_base_link" />
+    <child link="lidar_base_link" />
+    <origin xyz="0 0 0" rpy="0 0 0" />
+  </joint>
+   <!-- Battery base link -->
+  <xacro:base link_name="battery_base_link" base_prop="${battery_base_props}" mesh="${battery_base_props['base']['mesh']}" >
+    <origin xyz="0.035 0 0.0815" rpy="0 ${pi} 0" />
+  </xacro:base>
+  <!-- Joint to connect second_story with base_link -->
+  <joint name="battery_base_joint" type="fixed">
+    <parent link="base_link"/>
+    <child link="battery_base_link" />
     <origin xyz="0 0 0" rpy="0 0 0" />
   </joint>
   <!-- Caster Wheel -->
-  <xacro:caster_wheel reflect="-1"
-                      use_fixed="$(arg use_fixed_caster)"
-                      wheel_props="${caster_wheel_props}">
+  <xacro:caster_wheel wheel_props="${caster_wheel_props}">
   </xacro:caster_wheel>
   <!-- Wheels -->
   <xacro:wheel prefix="right" reflect="-1"
                       wheel_props="${wheel_props}"
-                      base_props="${base_props}" >
+                      motor_props="${motor_props}" >
   </xacro:wheel>
   <xacro:wheel prefix="left" reflect="1"
                       wheel_props="${wheel_props}"
-                      base_props="${base_props}" >
+                      motor_props="${motor_props}" >
   </xacro:wheel>
   <!-- Motors -->
@@ -63,5 +73,5 @@
   </xacro:motor>
   <!-- Sensors -->
-  <xacro:laser prefix="rplidar" parent_link="second_base_link"
+  <xacro:laser prefix="rplidar" parent_link="lidar_base_link"
                    sensor_prop="${sensor_prop}">
   </xacro:laser>

File: andino_description/urdf/include/andino_caster_macro.urdf.xacro (robot description, xacro)
@@ -5,8 +5,5 @@
 -->
 <!-- ===================== Caster xacro =========================================
-  Xacro to create caster links and the respective joints.
   params:
-  - reflect [1/-1]: value to set the side of the caster;
-  - use_fixed [bool]: wheter to use a fixed model or not
   - wheel_props [dictionary]: wheel properties;
   - base_props [dictionary]: base link properties;
@@ -16,117 +13,15 @@
 <!-- Caster wheel link & joint macro -->
   <xacro:macro name="caster_wheel"
-                params="reflect use_fixed wheel_props locationright:=${0} scale:=''">
-    <link name="caster_base_link">
-      <xacro:box_inertia  m="${wheel_props['base']['mass']}"
-                          x="${wheel_props['base']['size']['x']}"
-                          y="${wheel_props['base']['size']['y']}"
-                          z="${wheel_props['base']['size']['z']}"
-                          o_xyz="0.0 0.0 ${-wheel_props['base']['size']['z']/2.0}"
+                params="wheel_props scale:=''">
+    <link name="caster_link">
+      <xacro:box_inertia  m="${wheel_props['wheel']['mass']}"
+                          x="${wheel_props['wheel']['size']['x']}"
+                          y="${wheel_props['wheel']['size']['y']}"
+                          z="${wheel_props['wheel']['size']['z']}"
+                          o_xyz="0.0 0.0 ${-wheel_props['wheel']['size']['z']/2.0}"
                           o_rpy="0.0 0.0 0.0" />
-      <xacro:if value="${wheel_props['base']['mesh'] != '' }" >
-        <visual>
-          <origin xyz="0 0 ${-wheel_props['base']['size']['z']/2.0}" rpy="0 0 0" />
-          <geometry>
-            <xacro:if value="${scale != '' }" >
-              <mesh filename="package://andino_description/meshes/${robot_name}/${wheel_props['base']['mesh']}" scale="${scale}"/>
-            </xacro:if>
-            <xacro:if value="${scale == '' }" >
-              <mesh filename="package://andino_description/meshes/${robot_name}/${wheel_props['base']['mesh']}" />
-            </xacro:if>
-          </geometry>
-          <material name="silver"/>
-        </visual>
-      </xacro:if>
-      <xacro:if value="${wheel_props['base']['mesh'] == '' }" >
-        <visual>
-          <origin xyz="0 0 ${-wheel_props['base']['size']['z']/2.0}" rpy="0 0 0" />
-          <geometry>
-            <box size="${wheel_props['base']['size']['x']} ${wheel_props['base']['size']['y']} ${wheel_props['base']['size']['z']}" />
-          </geometry>
-          <material name="red"/>
-        </visual>
-      </xacro:if>
-      <collision>
-        <origin xyz="0 0 ${-wheel_props['base']['size']['z']/2.0}" rpy="0 0 0" />
-        <geometry>
-          <box size="${wheel_props['base']['size']['x']} ${wheel_props['base']['size']['y']} ${wheel_props['base']['size']['z']}" />
-        </geometry>
-      </collision>
-    </link>
-    <joint name="caster_base_joint" type="fixed">
-      <origin xyz="${wheel_props['base']['dx']} ${-wheel_props['base']['dy'] * locationright} ${wheel_props['base']['dz']}"
-              rpy="0 0 0" />
-      <parent link="base_link" />
-      <child link="caster_base_link" />
-      <axis xyz="0 0 1" />
-      <dynamics damping="0.01" friction="0.0"/>
-    </joint>
-    <!-- caster hub -->
-    <link name="caster_rotation_link">
-      <xacro:box_inertia  m="${wheel_props['hub']['mass']}"
-                          x="${wheel_props['hub']['size']['x']}"
-                          y="${wheel_props['hub']['size']['y']}"
-                          z="${wheel_props['hub']['size']['z']}"
-                          o_xyz="0.0 0.0 ${-wheel_props['hub']['size']['z']/2.0}"
-                          o_rpy="0.0 0.0 0.0" />
-      <xacro:if value="${wheel_props['hub']['mesh'] != '' }" >
-        <visual>
-          <origin xyz="0 0 ${-wheel_props['hub']['size']['z']/2.0}" rpy="0 0 0" />
-          <geometry>
-            <xacro:if value="${scale != '' }" >
-              <mesh filename="package://andino_description/meshes/${robot_name}/${wheel_props['hub']['mesh']}" scale="${scale}"/>
-            </xacro:if>
-            <xacro:if value="${scale == '' }" >
-              <mesh filename="package://andino_description/meshes/${robot_name}/${wheel_props['hub']['mesh']}" />
-            </xacro:if>
-          </geometry>
-          <material name="silver"/>
-        </visual>
-      </xacro:if>
-      <xacro:if value="${wheel_props['hub']['mesh'] == '' }" >
-        <visual>
-          <origin xyz="0 0 ${-wheel_props['hub']['size']['z']/2.0}" rpy="0 0 0" />
-          <geometry>
-            <box size="${wheel_props['hub']['size']['x']} ${wheel_props['hub']['size']['y']} ${wheel_props['hub']['size']['z']}" />
-          </geometry>
-          <material name="red"/>
-        </visual>
-      </xacro:if>
-      <collision>
-        <origin xyz="0 0 ${-wheel_props['hub']['size']['z']/2.0}" rpy="0 0 0" />
-        <geometry>
-          <box size="${wheel_props['hub']['size']['x']} ${wheel_props['hub']['size']['y']} ${wheel_props['hub']['size']['z']}" />
-        </geometry>
-      </collision>
-    </link>
-    <xacro:if value="${use_fixed}">
-      <joint name="caster_rotation_joint" type="fixed">
-        <origin xyz="${wheel_props['hub']['dx']} ${-wheel_props['hub']['dy'] * locationright} ${wheel_props['hub']['dz']}"
-                rpy="0 0 0" />
-        <parent link="base_link" />
-        <child link="caster_rotation_link" />
-        <axis xyz="0 0 1" />
-        <dynamics damping="0.01" friction="0.0"/>
-      </joint>
-    </xacro:if>
-    <xacro:unless value="${use_fixed}">
-      <joint name="caster_rotation_joint" type="continuous">
-        <origin xyz="${wheel_props['hub']['dx']} ${-wheel_props['hub']['dy'] * locationright} ${wheel_props['hub']['dz']}"
-                rpy="0 0 0" />
-        <parent link="base_link" />
-        <child link="caster_rotation_link" />
-        <axis xyz="0 0 1" />
-        <dynamics damping="0.01" friction="0.0"/>
-      </joint>
-    </xacro:unless>
-    <!-- caster wheel -->
-    <link name="caster_wheel_link">
-      <xacro:cylinder_inertia m="${wheel_props['wheel']['mass']}"
-                              r="${wheel_props['wheel']['radius']}"
-                              l="${wheel_props['wheel']['length']}">
-      </xacro:cylinder_inertia>
       <xacro:if value="${wheel_props['wheel']['mesh'] != '' }" >
         <visual>
-          <origin xyz="0 0 0" rpy="0 0 0" />
+          <origin xyz="0 0 0" rpy="${pi} 0 ${pi/2}" />
           <geometry>
             <xacro:if value="${scale != '' }" >
@@ -137,12 +32,12 @@
             </xacro:if>
           </geometry>
-          <material name="black"/>
+          <material name="silver"/>
         </visual>
       </xacro:if>
       <xacro:if value="${wheel_props['wheel']['mesh'] == '' }" >
         <visual>
-          <origin xyz="0 0 0" rpy="${pi/2} 0 0" />
+          <origin xyz="0 0 ${-wheel_props['wheel']['size']['z']/2.0}" rpy="0 0 0" />
           <geometry>
-            <cylinder length="${wheel_props['wheel']['length']}" radius="${wheel_props['wheel']['radius']}" />
+            <box size="${wheel_props['wheel']['size']['x']} ${wheel_props['wheel']['size']['y']} ${wheel_props['wheel']['size']['z']}" />
           </geometry>
           <material name="red"/>
@@ -150,28 +45,18 @@
       </xacro:if>
       <collision>
-        <origin xyz="0 0 0" rpy="${pi/2} 0 0" />
+        <origin xyz="0 0 ${-wheel_props['wheel']['size']['z']/2.0}" rpy="0 0 0" />
         <geometry>
-          <cylinder length="${wheel_props['wheel']['length']}" radius="${wheel_props['wheel']['radius']}" />
+          <box size="${wheel_props['wheel']['size']['x']} ${wheel_props['wheel']['size']['y']} ${wheel_props['wheel']['size']['z']}" />
         </geometry>
       </collision>
     </link>
-    <xacro:if value="${use_fixed}">
-      <joint name="caster_wheel_joint" type="fixed">
-        <origin xyz="${wheel_props['wheel']['dx']} ${-wheel_props['wheel']['dy'] * locationright} ${wheel_props['wheel']['dz']}"
-                rpy="0 0 0" />
-        <parent link="caster_rotation_link" />
-        <child link="caster_wheel_link" />
-        <axis xyz="0 1 0" />
-      </joint>
-    </xacro:if>
-    <xacro:unless value="${use_fixed}">
-      <joint name="caster_wheel_joint" type="continuous">
-        <origin xyz="${wheel_props['wheel']['dx']} ${-wheel_props['wheel']['dy'] * locationright} ${wheel_props['wheel']['dz']}"
-                rpy="0 0 0" />
-        <parent link="caster_rotation_link" />
-        <child link="caster_wheel_link" />
-        <axis xyz="0 1 0" />
-      </joint>
-    </xacro:unless>
+    <joint name="caster_base_joint" type="fixed">
+      <origin xyz="${wheel_props['wheel']['dx']} ${wheel_props['wheel']['dy']} ${wheel_props['wheel']['dz']}"
+              rpy="0 0 0" />
+      <parent link="base_link" />
+      <child link="caster_link" />
+      <axis xyz="0 0 1" />
+      <dynamics damping="0.01" friction="0.0"/>
+    </joint>
   </xacro:macro>
 </robot>

File: andino_description/urdf/include/common_macros.urdf.xacro (robot description, xacro)
@@ -6,15 +6,16 @@
   - reflect [1/-1]: value to set the side of the wheel;
   - wheel_props [dictionary]: wheel properties;
-  - base_props [dictionary]: base link properties;
+  - motor_props [dictionary]: motor link properties;
   - mesh [string]: file name of the wheel mesh;
     - DEFAULT Value -> Empty string
 -->
   <xacro:macro name="wheel"
-               params="prefix reflect wheel_props base_props ">
+               params="prefix reflect wheel_props motor_props ">
   <xacro:property name="pos_x_joint"
-     value="${(base_props['base']['x_size']/2) - wheel_props['x_offset']}"/>
+     value="${(motor_props['x_offset']) + wheel_props['x_offset']}"/>
   <xacro:property name="pos_y_joint"
-    value="${(base_props['base']['y_size']/2) + wheel_props['y_offset'] + (wheel_props['length']/2)}"/>
-  <xacro:property name="pos_z_joint" value="${wheel_props['z_offset']}"/>
+    value="${(motor_props['y_offset']) + wheel_props['y_offset']}"/>
+  <xacro:property name="pos_z_joint"
+    value="${(motor_props['z_offset']) + wheel_props['z_offset']}"/>
     <link name="${prefix}_wheel">
     <xacro:if value="${wheel_props['mesh'] != '' }" >
@@ -73,8 +74,6 @@
   <xacro:macro name="motor"
                params="prefix reflect motor_props base_props ">
-  <xacro:property name="pos_x_joint"
-     value="${(base_props['base']['x_size']/2) - motor_props['x_offset']}"/>
-  <xacro:property name="pos_y_joint"
-    value="${(base_props['base']['y_size']/2) + motor_props['y_offset'] + (motor_props['y_size']/2)}"/>
+  <xacro:property name="pos_x_joint" value="${motor_props['x_offset']}"/>
+  <xacro:property name="pos_y_joint" value="${motor_props['y_offset']}"/>
   <xacro:property name="pos_z_joint" value="${motor_props['z_offset']}"/>
     <link name="${prefix}_motor">
@@ -162,5 +161,5 @@
     </xacro:if>
     <collision>
-      <origin xyz="0.0 0.0 0.0" rpy="0.0 0.0 0.0"/>
+      <origin xyz="-0.02 0.0 ${base_prop['base']['z_size']/2.0}" rpy="0.0 0.0 0.0"/>
       <geometry>
         <box size="${base_prop['base']['x_size']} ${base_prop['base']['y_size']} ${base_prop['base']['z_size']}"/>
